Commit message: pybullet

File: testing/pybullet_ik_text/niryo.urdf (robot description, URDF)
Before this commit: robot NiryoOne, 14 links, 13 joints
Links:
- link robot_base: geometry collision mesh filename=file://C:/Users/ANILM/Downloads/niryo_urdf/niryo_robot_base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; visual mesh filename=file://C:/Users/ANILM/Downloads/niryo_urdf/niryo_visible_vi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
Joints:
- joint Joint: origin xyz=-0.374921 0.300036 0.095000 rpy=-3.141593 3.141593 -3.141593 -> xyz=0.000079 0.006036 0.044000 rpy=-3.141593 3.141593 -3.141593
